Commit message: * Add optimization method to solve inverse kinematics

File: urdf/ur10e.urdf (robot description, URDF)
Before this commit: robot /Users/hu/Downloads/UR10e.urdf, 21 links, 20 joints
Joints:
- joint shoulder_lift_joint: limit lower=-6.28319 upper=6.28319 effort=330 velocity=3.14 -> lower=-3.14159 upper=3.14159 effort=330 velocity=3.14
- joint shoulder_pan_joint: limit lower=-6.28319 upper=6.28319 effort=330 velocity=3.14 -> lower=-3.14159 upper=3.14159 effort=330 velocity=3.14
- joint wrist_1_joint: limit lower=-6.28319 upper=6.28319 effort=54 velocity=6.28 -> lower=-3.14159 upper=3.14159 effort=54 velocity=6.28
- joint wrist_2_joint: limit lower=-6.28319 upper=6.28319 effort=54 velocity=6.28 -> lower=-3.14159 upper=3.14159 effort=54 velocity=6.28
- joint wrist_3_joint: limit lower=-6.28319 upper=6.28319 effort=54 velocity=6.28 -> lower=-3.14159 upper=3.14159 effort=54 velocity=6.28
